File: Schematic/t10_schem.sch (EAGLE design)
At the start: 31 parts, among them IC1 MIC5219BM5, Q1 1109200 Hz, Q2 MOSFET-NCHANNEL2N7000, Q3 MOSFET-NCHANNEL2N7000, Q4 MOSFET-NCHANNEL2N7000, U1 ATMEGA328P_PDIP, U2 LM386

Commit message: official preliminary schematic
v1.01
Parts:
- removed IC1: MIC5219BM5, v-reg-micrel:MIC5219BM5
- removed LED1: (no value), led:LED
- removed Q2, Q3, Q4: MOSFET-NCHANNEL2N7000, SparkFun-DiscreteSemi:MOSFET-NCHANNEL2N7000
- removed R10, R11: 10k, resistor:R-US_M0805
- removed R5, R7, R8, R9: 10K, resistor:R-US_M0805
- removed SP1: SMS-1308MS-2-R, speaker:SMS-1308MS-2-R
- added D1: 1N4004, diode:1N4004
- added J2: DCJ0202, con-jack:DCJ0202
- added S1: 1, SparkFun-Electromechanical:SWITCH-SPDT-SMD-A
- added SPEAKERHDR: 22-23-2021, con-molex:22-23-2021
- C3, C4: value 0.1uF -> 100nF
- C8, C9: value (none) -> 100pF
- J1: value (none) -> 1
Connections:
- removed net +3V3: C9.1, IC1.OUT, J1.3
- removed net N$10: LED1.A, R10.1
- removed net N$16: LED1.C, Q4.D
- removed net N$17: Q4.G, R11.1
- removed net N$2 (its old number): C2.1, U1.PB7(XTAL2/TOSC2)
- removed net SCL_3V: Q3.S, R7.1
- removed net SDA_3V: Q2.S, R5.1
- new net N$1: C2.1, Q1.1, U1.PB7(XTAL2/TOSC2)
- net 3.3V: now also J1.3; no longer Q2.G, Q3.G, R10.2, R11.2, R5.2, R7.2
- net GND: now also J2.2, J2.3, SPEAKERHDR-2.S; no longer IC1.GND, Q1.1, Q4.S, SP1.2
- net N$13: now also D1.A, J2.1; no longer Q2.D, R8.1
- net N$14: now also SPEAKERHDR-1.S; no longer SP1.1
- net N$15: now also D1.C, S1.P; no longer Q3.D, R9.1
- net SCL_5.0V: now also J1.5; no longer J1.4
- net SDA_5.0V: now also J1.4; no longer J1.5
- net SM1-CLK: now also SM1-5.1; no longer SM1-3.1
- net SM1-DAT: now also SM1-3.1; no longer SM1-5.1
- net VIN: now also C9.1, S1.O, U1.AVCC, U1.VCC; no longer IC1.EN, IC1.IN, R8.2, R9.2
Other:
- note added: "2"
- note added: "5V 12W DC power supply"
- note added: "Header connection for TCS3472 RGB sensor"
- note added: "Team T10: Carmen Ciobanu, Deborah Denhart, Jeremiah Scott, Nick Lynch-Jonely"
- note added: "v1.01"
- note removed: "0.1"
- note removed: "Actual Color Sensor"
- note removed: "LED strip"
- note removed: "Power Circuit"
- note removed: "STILL MISSING:"
- note removed: "This is supposed to be the Vregulator built in to the color sensor board"
- note removed: "This is the LED for the sensor board"
- note removed: "This is the jumper header for the color sensor daughter board"
- note removed: "This is the level shifter from 5V to 3V for the sensor"
- note removed: "whatever other pin outs MCU needs"
- moved on the sheet: C1, C2, C3, C4, C5, C6, C7, C8, C9, J1, Q1, R1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
